File: RaspBle.sch (EAGLE design)
At the start: 17 parts, among them U1 RN4020, U2 MCP1703T-3302E/CB

Commit message: Rev A and pdf files added
Other:
- note added: "A"
- note removed: "1.0"
Changed lines of the file:
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@@
 <text x="213.36" y="111.76" size="1.778" layer="97">Red led. UART console data.</text>
 <text x="213.36" y="101.6" size="1.778" layer="97">Blue led. Module is awake and active.</text>
-<text x="254" y="7.62" size="2.54" layer="97" align="center-left">1.0</text>
+<text x="254" y="7.62" size="2.54" layer="97" align="center-left">A</text>
 </plain>
 <instances>
